File: micorcontroller/Hardware/MotherboardV4/Power.kicad_sch (KiCad schematic)
At the start: 66 parts, among them IC12 LM2596SX-5.0_NOPB, IC3 MCP1826S-5002E_DB, IC71 LMR51430YFDDCR, J2 MS3112E8-4P, Q1 FDN304P, U3 LM2904AVQDRQ1

Commit message: some moving around
Parts:
- removed IC12: LM2596SX-5.0_NOPB, KTT0005B, symbol SamacSys_Parts:LM2596SX-5.0_NOPB
- removed IC71: LMR51430YFDDCR, symbol SamacSys_Parts:LMR51430YFDDCR
- removed R20: 49.9, Resistor_SMD:R_0603_1608Metric_Pad0.98x0.95mm_HandSolder, symbol Device:R_Small
- C39: value 0.1u -> 22u; footprint Capacitor_SMD:C_0402_1005Metric_Pad0.74x0.62mm_HandSolder -> Capacitor_SMD:C_0805_2012Metric_Pad1.18x1.45mm_HandSolder
- C66: value DNP -> 12p
- L1: symbol SamacSys_Parts:74439346068 -> Device:L_Small
- R19: value 0 -> DNP
- R24: value 10.2k -> 10k
- R47: value 53.6k -> 64.9k
Connections:
- net 5VBuck: now also C66.1, R47.2
Other:
- moved on the sheet: C11, C14, C17, C22, C23, C25, C38, C66, R24, R47
