File: micorcontroller/Hardware/MotherboardV4/Heater.kicad_sch (KiCad schematic)
At the start: 48 parts

Commit message: added uplink
Parts:
- C66, C67, C68, C69, C70, C71, C72, C73, C74, C75, C76, C77: symbol Device:C -> SymbolsBalloonv4:C
- F1, F2, F3, F4, F5, F6, F7, F8: symbol Device:Fuse_Small -> SymbolsBalloonv4:Fuse_Small
- H0, H1, H2, H3, H4, H5, H6, H7: symbol SamacSys_Parts:ITS4200S-ME-O -> SymbolsBalloonv4:ITS4200S-ME-O
- H1-0: symbol SamacSys_Parts:502352-0400 -> SymbolsBalloonv4:502352-0400
- H3-0: symbol SamacSys_Parts:502352-1210 -> SymbolsBalloonv4:502352-1210
- JHEAT0: symbol Connector_Generic:Conn_01x02 -> SymbolsBalloonv4:Conn_01x02
- R81, R82, R83, R87, R88, R89, R93, R94: symbol Device:Heater -> SymbolsBalloonv4:Heater
- R84, R85, R86, R90, R91, R92, R95, R96: symbol Device:R -> SymbolsBalloonv4:R
- Vshi0: symbol SamacSys_Parts:TXS0108EQPWRQ1 -> SymbolsBalloonv4:TXS0108EQPWRQ1
