File: micorcontroller/Hardware/MotherboardV4/Sensors.kicad_sch (KiCad schematic)
At the start: 53 parts

Commit message: changed debug to level based debug and started writing driver for FD-OEM Module
Other:
- moved on the sheet: C44, OP1B, R37, Vref1
Changed lines of the file:
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@@
 	)
 	(no_connect
-		(at 132.08 140.97)
+		(at 125.73 135.89)
 	)
 	(no_connect
-		(at 147.32 143.51)
+		(at 140.97 138.43)
 	)
 	(no_connect
-		(at 132.08 146.05)
+		(at 125.73 140.97)
 	)
 	(no_connect
@@
 	(wire
 		(pts
-			(xy 44.45 156.21) (xy 44.45 157.48)
+			(xy 48.26 157.48) (xy 48.26 158.75)
 		)
 		(stroke
@@
 	(wire
 		(pts
-			(xy 163.83 118.11) (xy 163.83 116.84)
+			(xy 217.17 119.38) (xy 217.17 118.11)
 		)
 		(stroke
@@
 	(wire
 		(pts
-			(xy 44.45 176.53) (xy 44.45 175.26)
+			(xy 48.26 177.8) (xy 48.26 176.53)
 		)
 		(stroke
@@
 	(wire
 		(pts
-			(xy 44.45 165.1) (xy 44.45 167.64)
+			(xy 48.26 166.37) (xy 48.26 168.91)
 		)
 		(stroke
@@
 	)
 	(arc
-		(start 81.2439 132.6404)
-		(mid 81.244 132.6596)
-		(end 81.2369 132.6487)
+		(start 81.2369 132.6487)
+		(mid 81.2388 132.6431)
+		(end 81.2439 132.6404)
 		(stroke
 			(width 0.08)
@@
 	)
 	(arc
-		(start 95.35 138.0726)
-		(mid 95.3708 138.0738)
-		(end 95.3605 138.0844)
+		(start 95.3605 138.0844)
+		(mid 95.3514 138.0815)
+		(end 95.35 138.0726)
 		(stroke
 			(width 0.08)
@@
 	)
 	(arc
-		(start 85.0546 136.1217)
-		(mid 85.0391 136.1162)
-		(end 85.0477 136.107)
+		(start 85.0477 136.107)
+		(mid 85.0601 136.1115)
+		(end 85.0546 136.1217)
 		(stroke
 			(width 0.08)
@@
 	)
 	(arc
-		(start 82.4029 136.7281)
-		(mid 82.4004 136.7249)
-		(end 82.4032 136.7206)
+		(start 82.4032 136.7206)
+		(mid 82.4025 136.7221)
+		(end 82.4029 136.7281)
 		(stroke
 			(width 0.08)
@@
 	)
 	(arc
-		(start 94.281 135.9581)
-		(mid 94.2805 135.9581)
-		(end 94.28 135.9518)
+		(start 94.28 135.9518)
+		(mid 94.2839 135.9543)
+		(end 94.281 135.9581)
 		(stroke
 			(width 0.08)
@@
 	)
 	(label "ntc+"
-		(at 44.45 166.37 0)
+		(at 48.26 167.64 0)
 		(fields_autoplaced yes)
 		(effects
@@
 	(hierarchical_label "3V3uC"
 		(shape input)
-		(at 44.45 156.21 90)
+		(at 48.26 157.48 90)
 		(fields_autoplaced yes)
 		(effects
@@
 	(hierarchical_label "3V3uC"
 		(shape input)
-		(at 163.83 109.22 90)
+		(at 217.17 110.49 90)
 		(fields_autoplaced yes)
 		(effects
@@
 	(symbol
 		(lib_id "SymbolsBalloonv4:Opamp_Dual")
-		(at 139.7 143.51 0)
+		(at 133.35 138.43 0)
 		(unit 2)
 		(exclude_from_sim no)
@@
 		(on_board yes)
 		(dnp no)
-		(fields_autoplaced yes)
 		(property "Reference" "OP1"
-			(at 139.7 133.35 0)
+			(at 134.112 132.334 0)
 			(effects
 				(font
@@
 		)
 		(property "Value" "TLV9002QDRQ1"
-			(at 139.7 135.89 0)
+			(at 133.35 130.81 0)
 			(effects
 				(font
 					(size 1.27 1.27)
 				)
+				(hide yes)
 			)
 		)
 		(property "Footprint" "SamacSys_Parts:SOIC127P600X175-8N"
-			(at 139.7 143.51 0)
+			(at 133.35 138.43 0)
 			(effects
 				(font
@@
 		)
 		(property "Datasheet" "~"
-			(at 139.7 143.51 0)
+			(at 133.35 138.43 0)
 			(effects
 				(font
@@
 		)
 		(property "Description" "Dual operational amplifier"
-			(at 139.7 143.51 0)
+			(at 133.35 138.43 0)
 			(effects
 				(font
@@
 		)
 		(property "Sim.Library" "${KICAD7_SYMBOL_DIR}/Simulation_SPICE.sp"
-			(at 139.7 143.51 0)
+			(at 133.35 138.43 0)
 			(effects
 				(font
@@
 		)
 		(property "Sim.Name" "kicad_builtin_opamp_dual"
-			(at 139.7 143.51 0)
+			(at 133.35 138.43 0)
 			(effects
 				(font
@@
 		)
 		(property "Sim.Device" "SUBCKT"
-			(at 139.7 143.51 0)
+			(at 133.35 138.43 0)
 			(effects
 				(font
@@
 		)
 		(property "Sim.Pins" "1=out1 2=in1- 3=in1+ 4=vee 5=in2+ 6=in2- 7=out2 8=vcc"
-			(at 139.7 143.51 0)
+			(at 133.35 138.43 0)
 			(effects
 				(font
@@
 	(symbol
 		(lib_id "SymbolsBalloonv4:GND")
-		(at 44.45 176.53 0)
+		(at 48.26 177.8 0)
 		(unit 1)
 		(exclude_from_sim no)
@@
 		(dnp no)
 		(property "Reference" "#PWR065"
-			(at 44.45 182.88 0)
+			(at 48.26 184.15 0)
 			(effects
 				(font
@@
 		)
 		(property "Value" "GND"
-			(at 44.577 180.9242 0)
+			(at 48.387 182.1942 0)
 			(effects
 				(font
@@
 		)
 		(property "Footprint" ""
-			(at 44.45 176.53 0)
+			(at 48.26 177.8 0)
 			(effects
 				(font
@@
 		)
 		(property "Datasheet" ""
-			(at 44.45 176.53 0)
+			(at 48.26 177.8 0)
 			(effects
 				(font
@@
 		)
 		(property "Description" "Power symbol creates a global label with name \"GND\" , ground"
-			(at 44.45 176.53 0)
+			(at 48.26 177.8 0)
 			(effects
 				(font
@@
 	(symbol
 		(lib_id "SymbolsBalloonv4:GND")
-		(at 163.83 118.11 0)
+		(at 217.17 119.38 0)
 		(unit 1)
 		(exclude_from_sim no)
@@
 		(dnp no)
 		(property "Reference" "#PWR073"
-			(at 163.83 124.46 0)
+			(at 217.17 125.73 0)
 			(effects
 				(font
@@
 		)
 		(property "Value" "GND"
-			(at 163.83 122.174 0)
+			(at 217.17 123.444 0)
 			(effects
 				(font
@@
 		)
 		(property "Footprint" ""
-			(at 163.83 118.11 0)
+			(at 217.17 119.38 0)
 			(effects
 				(font
@@
 		)
 		(property "Datasheet" ""
-			(at 163.83 118.11 0)
+			(at 217.17 119.38 0)
 			(effects
 				(font
@@
 		)
 		(property "Description" "Power symbol creates a global label with name \"GND\" , ground"
-			(at 163.83 118.11 0)
+			(at 217.17 119.38 0)
 			(effects
 				(font
@@
 					(size 1.27 1.27)
 				)
+				(hide yes)
 			)
 		)
@@
 	(symbol
 		(lib_id "SymbolsBalloonv4:D_Zener")
-		(at 44.45 171.45 270)
+		(at 48.26 172.72 270)
 		(unit 1)
 		(exclude_from_sim no)
@@
 		(dnp no)
 		(property "Reference" "Vref1"
-			(at 41.148 170.434 90)
+			(at 44.958 171.704 90)
 			(effects
 				(font
@@
 		)
 		(property "Value" "LM4040BIM3-3.0_NOPB"
-			(at 41.148 172.974 90)
+			(at 44.958 174.244 90)
 			(effects
 				(font
@@
 		)
 		(property "Footprint" "SamacSys_Parts:SOT95P237X112-3N"
-			(at 47.752 172.212 0)
+			(at 51.562 173.482 0)
 			(effects
 				(font
@@
 		)
 		(property "Datasheet" "~"
-			(at 44.45 171.45 0)
+			(at 48.26 172.72 0)
 			(effects
 				(font
@@
 		)
 		(property "Description" "Zener diode"
-			(at 40.64 181.61 0)
+			(at 44.45 182.88 0)
 			(effects
 				(font
@@
 		)
 		(property "Height" "1.12"
-			(at 39.37 190.5 0)
+			(at 43.18 191.77 0)
 			(effects
 				(font
@@
 		)
 		(property "Mouser Part Number" "926-LM4040BIM330NOPB"
-			(at 36.83 190.5 0)
+			(at 40.64 191.77 0)
 			(effects
 				(font
@@
 		)
 		(property "Mouser Price/Stock" "https://www.mouser.co.uk/ProductDetail/Texas-Instruments/LM4040BIM3-3.0-NOPB?qs=QbsRYf82W3FThDimo07Imw%3D%3D"
-			(at 34.29 190.5 0)
+			(at 38.1 191.77 0)
 			(effects
 				(font
@@
 		)
 		(property "Manufacturer_Name" "Texas Instruments"
-			(at 31.75 190.5 0)
+			(at 35.56 191.77 0)
 			(effects
 				(font
@@
 		)
 		(property "Manufacturer_Part_Number" "LM4040BIM3-3.0/NOPB"
-			(at 29.21 190.5 0)
+			(at 33.02 191.77 0)
 			(effects
 				(font
@@
 	(symbol
 		(lib_id "SymbolsBalloonv4:R")
-		(at 44.45 161.29 0)
+		(at 48.26 162.56 0)
 		(unit 1)
 		(exclude_from_sim no)
@@
 		(dnp no)
 		(property "Reference" "R37"
-			(at 38.608 161.29 90)
+			(at 42.418 162.56 90)
 			(effects
 				(font
@@
 		)
 		(property "Value" "270"
-			(at 40.64 161.798 90)
+			(at 44.45 163.068 90)
 			(effects
 				(font
@@
 		)
 		(property "Footprint" "Resistor_SMD:R_0603_1608Metric_Pad0.98x0.95mm_HandSolder"
-			(at 42.672 161.29 90)
+			(at 46.482 162.56 90)
 			(effects
 				(font
@@
 		)
 		(property "Datasheet" "~"
-			(at 44.45 161.29 0)
+			(at 48.26 162.56 0)
 			(effects
 				(font
@@
 		)
 		(property "Description" "Zdiode Cur limiter"
-			(at 28.448 161.798 0)
+			(at 32.258 163.068 0)
 			(show_name yes)
 			(effects
@@
 	(symbol
 		(lib_id "SymbolsBalloonv4:C")
-		(at 163.83 113.03 0)
+		(at 217.17 114.3 0)
 		(unit 1)
 		(exclude_from_sim no)
@@
 		(dnp no)
 		(property "Reference" "C44"
-			(at 166.751 111.8616 0)
+			(at 220.091 113.1316 0)
 			(effects
 				(font
@@
 		)
 		(property "Value" "10u"
-			(at 166.751 114.173 0)
+			(at 220.091 115.443 0)
 			(effects
 				(font
@@
 		)
 		(property "Footprint" "Capacitor_SMD:C_0805_2012Metric_Pad1.18x1.45mm_HandSolder"
-			(at 164.7952 116.84 0)
+			(at 218.1352 118.11 0)
 			(effects
 				(font
@@
 		)
 		(property "Datasheet" "~"
-			(at 163.83 113.03 0)
+			(at 217.17 114.3 0)
 			(effects
 				(font
@@
 		)
 		(property "Description" "Unpolarized capacitor"
-			(at 163.83 113.03 0)
+			(at 217.17 114.3 0)
 			(effects
 				(font
