File: micorcontroller/Hardware/MotherboardV4.1/Ethernet.kicad_sch (KiCad schematic)
At the start: 48 parts, among them J501 J1B1211CCD, Y501 ECS-250-6-33B2-CTP-TR

Commit message: cleanup
Parts:
- R511, R514: value 330 -> 510
Changed lines of the file:
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@@
 			)
 		)
-		(property "Value" "330"
+		(property "Value" "510"
 			(at 227.33 126.365 90)
 			(effects
@@
 			)
 		)
-		(property "Value" "330"
+		(property "Value" "510"
 			(at 228.6 136.525 90)
 			(effects
