File: micorcontroller/Hardware/MotherboardV4.1/Heater.kicad_sch (KiCad schematic)
At the start: 60 parts, among them J0 0, Q601 IRLML6344TRPBF, Q602 IRLML6344TRPBF, Q603 IRLML6344TRPBF, Q604 IRLML6344TRPBF, Q605 IRLML6344TRPBF, Q606 IRLML6344TRPBF, Q607 IRLML6344TRPBF, Q608 IRLML6344TRPBF

Commit message: cleanup
Parts:
- R607, R608, R609, R610, R611, R613, R619, R620: value 100 -> 220
Changed lines of the file:
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@@
 			)
 		)
-		(property "Value" "100"
+		(property "Value" "220"
 			(at 84.074 161.544 90)
 			(effects
@@
 			)
 		)
-		(property "Value" "100"
+		(property "Value" "220"
 			(at 40.894 161.544 90)
 			(effects
@@
 			)
 		)
-		(property "Value" "100"
+		(property "Value" "220"
 			(at 226.314 114.554 90)
 			(effects
@@
 			)
 		)
-		(property "Value" "100"
+		(property "Value" "220"
 			(at 133.604 110.744 90)
 			(effects
@@
 			)
 		)
-		(property "Value" "100"
+		(property "Value" "220"
 			(at 273.304 114.554 90)
 			(effects
@@
 			)
 		)
-		(property "Value" "100"
+		(property "Value" "220"
 			(at 87.884 110.744 90)
 			(effects
@@
 			)
 		)
-		(property "Value" "100"
+		(property "Value" "220"
 			(at 181.864 113.284 90)
 			(effects
@@
 			)
 		)
-		(property "Value" "100"
+		(property "Value" "220"
 			(at 39.624 110.744 90)
 			(effects
