File: micorcontroller/Hardware/MotherboardV4.1/Power.kicad_sch (KiCad schematic)
At the start: 46 parts, among them IC201 INA240A3EDRQ1, J201 0, J202 MS3112E8-4P

Commit message: cleanup
Parts:
- R205: value 12k -> 12.4k 1%
- R206: value 500 -> 510
Changed lines of the file:
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@@
 			)
 		)
-		(property "Value" "12k"
+		(property "Value" "12.4k 1%"
 			(at 120.65 90.805 90)
 			(effects
@@
 			)
 		)
-		(property "Value" "500"
+		(property "Value" "510"
 			(at 132.08 90.17 90)
 			(effects
