File: micorcontroller/Hardware/MotherboardV4.1/Prozessor.kicad_sch (KiCad schematic)
At the start: 45 parts, among them Y301 ABM8G-12.000MHZ-4Y-T3

Commit message: cleanup
Parts:
- R0: value 500 -> 510
- R307, R308, R309, R310: value 4.7k -> 5.1k 1%
Changed lines of the file:
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@@
 			)
 		)
-		(property "Value" "4.7k"
+		(property "Value" "5.1k 1%"
 			(at 53.848 94.996 90)
 			(effects
@@
 			)
 		)
-		(property "Value" "4.7k"
+		(property "Value" "5.1k 1%"
 			(at 46.228 96.266 90)
 			(effects
@@
 			)
 		)
-		(property "Value" "500"
+		(property "Value" "510"
 			(at 255.27 110.49 90)
 			(effects
@@
 			)
 		)
-		(property "Value" "4.7k"
+		(property "Value" "5.1k 1%"
 			(at 57.658 136.906 90)
 			(effects
@@
 			)
 		)
-		(property "Value" "4.7k"
+		(property "Value" "5.1k 1%"
 			(at 50.038 138.176 90)
 			(effects
