File: motherboard/Hardware/MotherboardV4.1/Sensors.kicad_sch (KiCad schematic)
At the start: 33 parts, among them J401 0

Commit message: changed opamp
Parts:
- OP401: value TLV9002QDRQ1 -> OPA2377AID
Changed lines of the file:
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@@
 	)
 	(arc
-		(start 90.1269 103.4387)
-		(mid 90.1288 103.4331)
-		(end 90.1339 103.4304)
+		(start 90.1339 103.4304)
+		(mid 90.134 103.4496)
+		(end 90.1269 103.4387)
 		(stroke
 			(width 0.08)
@@
 	)
 	(arc
-		(start 104.2505 108.8744)
-		(mid 104.2414 108.8715)
-		(end 104.24 108.8626)
+		(start 104.24 108.8626)
+		(mid 104.2608 108.8638)
+		(end 104.2505 108.8744)
 		(stroke
 			(width 0.08)
@@
 	)
 	(arc
-		(start 93.9377 106.897)
-		(mid 93.9501 106.9015)
-		(end 93.9446 106.9117)
+		(start 93.9446 106.9117)
+		(mid 93.9291 106.9062)
+		(end 93.9377 106.897)
 		(stroke
 			(width 0.08)
@@
 	)
 	(arc
-		(start 91.2932 107.5106)
-		(mid 91.2925 107.5121)
-		(end 91.2929 107.5181)
+		(start 91.2929 107.5181)
+		(mid 91.2904 107.5149)
+		(end 91.2932 107.5106)
 		(stroke
 			(width 0.08)
@@
 	)
 	(arc
-		(start 103.17 106.7418)
-		(mid 103.1741 106.7445)
-		(end 103.171 106.7481)
+		(start 103.171 106.7481)
+		(mid 103.1705 106.7481)
+		(end 103.17 106.7418)
 		(stroke
 			(width 0.08)
@@
 			)
 		)
-		(property "Value" "TLV9002QDRQ1"
+		(property "Value" "OPA2377AID"
 			(at 155.702 138.684 0)
 			(effects
@@
 			)
 		)
-		(property "Value" "TLV9002QDRQ1"
+		(property "Value" "OPA2377AID"
 			(at 142.24 101.6 0)
 			(effects
@@
 			)
 		)
-		(property "Value" "TLV9002QDRQ1"
+		(property "Value" "OPA2377AID"
 			(at 116.84 144.78 0)
 			(effects

Commit message: refined thermal controller
Parts:
- C404: value DNP -> 10n; now fitted; now in the parts list
- J5: renamed from R414; value 1k -> 0
- J6: renamed from R416; value 1k -> 0
- J7: renamed from R415; value 1k -> 0
Changed lines of the file:
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@@
 	)
 	(arc
-		(start 90.1339 103.4304)
-		(mid 90.134 103.4496)
-		(end 90.1269 103.4387)
+		(start 90.1269 103.4387)
+		(mid 90.1288 103.4331)
+		(end 90.1339 103.4304)
 		(stroke
 			(width 0.08)
@@
 	)
 	(arc
-		(start 104.24 108.8626)
-		(mid 104.2608 108.8638)
-		(end 104.2505 108.8744)
+		(start 104.2505 108.8744)
+		(mid 104.2414 108.8715)
+		(end 104.24 108.8626)
 		(stroke
 			(width 0.08)
@@
 	)
 	(arc
-		(start 93.9446 106.9117)
-		(mid 93.9291 106.9062)
-		(end 93.9377 106.897)
+		(start 93.9377 106.897)
+		(mid 93.9501 106.9015)
+		(end 93.9446 106.9117)
 		(stroke
 			(width 0.08)
@@
 	)
 	(arc
-		(start 91.2929 107.5181)
-		(mid 91.2904 107.5149)
-		(end 91.2932 107.5106)
+		(start 91.2932 107.5106)
+		(mid 91.2925 107.5121)
+		(end 91.2929 107.5181)
 		(stroke
 			(width 0.08)
@@
 	)
 	(arc
-		(start 103.171 106.7481)
-		(mid 103.1705 106.7481)
-		(end 103.17 106.7418)
+		(start 103.17 106.7418)
+		(mid 103.1741 106.7445)
+		(end 103.171 106.7481)
 		(stroke
 			(width 0.08)
@@
 		(on_board yes)
 		(dnp no)
-		(property "Reference" "R414"
+		(property "Reference" "J5"
 			(at 104.14 132.334 90)
 			(effects
@@
 			)
 		)
-		(property "Value" "1k"
+		(property "Value" "0"
 			(at 104.394 136.398 90)
 			(effects
@@
 			(project "BalloonMotherboardV4.1"
 				(path "/a70d325c-f83f-4714-a2b6-4ef8919d016e/5e9e7f42-9819-4074-87ce-68c089720394"
-					(reference "R414")
+					(reference "J5")
 					(unit 1)
 				)
@@
 		(on_board yes)
 		(dnp no)
-		(property "Reference" "R416"
+		(property "Reference" "J6"
 			(at 104.394 137.922 90)
 			(effects
@@
 			)
 		)
-		(property "Value" "1k"
+		(property "Value" "0"
 			(at 104.394 141.732 90)
 			(effects
@@
 			(project "BalloonMotherboardV4.1"
 				(path "/a70d325c-f83f-4714-a2b6-4ef8919d016e/5e9e7f42-9819-4074-87ce-68c089720394"
-					(reference "R416")
+					(reference "J6")
 					(unit 1)
 				)
@@
 		(on_board yes)
 		(dnp no)
-		(property "Reference" "R415"
+		(property "Reference" "J7"
 			(at 132.334 135.382 90)
 			(effects
@@
 			)
 		)
-		(property "Value" "1k"
+		(property "Value" "0"
 			(at 132.334 139.192 90)
 			(effects
@@
 			(project "BalloonMotherboardV4.1"
 				(path "/a70d325c-f83f-4714-a2b6-4ef8919d016e/5e9e7f42-9819-4074-87ce-68c089720394"
-					(reference "R415")
+					(reference "J7")
 					(unit 1)
 				)
@@
 		(unit 1)
 		(exclude_from_sim no)
-		(in_bom no)
+		(in_bom yes)
 		(on_board yes)
-		(dnp yes)
+		(dnp no)
 		(fields_autoplaced yes)
 		(property "Reference" "C404"
@@
 			)
 		)
-		(property "Value" "DNP"
+		(property "Value" "10n"
 			(at 88.9 146.0499 0)
 			(effects

Commit message: working on thermal
Changed lines of the file:
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@@
 	)
 	(arc
-		(start 90.1269 103.4387)
-		(mid 90.1288 103.4331)
-		(end 90.1339 103.4304)
+		(start 90.1339 103.4304)
+		(mid 90.134 103.4496)
+		(end 90.1269 103.4387)
 		(stroke
 			(width 0.08)
@@
 	)
 	(arc
-		(start 104.2505 108.8744)
-		(mid 104.2414 108.8715)
-		(end 104.24 108.8626)
+		(start 104.24 108.8626)
+		(mid 104.2608 108.8638)
+		(end 104.2505 108.8744)
 		(stroke
 			(width 0.08)
@@
 	)
 	(arc
-		(start 93.9377 106.897)
-		(mid 93.9501 106.9015)
-		(end 93.9446 106.9117)
+		(start 93.9446 106.9117)
+		(mid 93.9291 106.9062)
+		(end 93.9377 106.897)
 		(stroke
 			(width 0.08)
@@
 	)
 	(arc
-		(start 91.2932 107.5106)
-		(mid 91.2925 107.5121)
-		(end 91.2929 107.5181)
+		(start 91.2929 107.5181)
+		(mid 91.2904 107.5149)
+		(end 91.2932 107.5106)
 		(stroke
 			(width 0.08)
@@
 	)
 	(arc
-		(start 103.17 106.7418)
-		(mid 103.1741 106.7445)
-		(end 103.171 106.7481)
+		(start 103.171 106.7481)
+		(mid 103.1705 106.7481)
+		(end 103.17 106.7418)
 		(stroke
 			(width 0.08)

Commit message: worked on thermals
Changed lines of the file:
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@@
 	)
 	(arc
-		(start 90.1339 103.4304)
-		(mid 90.134 103.4496)
-		(end 90.1269 103.4387)
+		(start 90.1269 103.4387)
+		(mid 90.1288 103.4331)
+		(end 90.1339 103.4304)
 		(stroke
 			(width 0.08)
@@
 	)
 	(arc
-		(start 104.24 108.8626)
-		(mid 104.2608 108.8638)
-		(end 104.2505 108.8744)
+		(start 104.2505 108.8744)
+		(mid 104.2414 108.8715)
+		(end 104.24 108.8626)
 		(stroke
 			(width 0.08)
@@
 	)
 	(arc
-		(start 93.9446 106.9117)
-		(mid 93.9291 106.9062)
-		(end 93.9377 106.897)
+		(start 93.9377 106.897)
+		(mid 93.9501 106.9015)
+		(end 93.9446 106.9117)
 		(stroke
 			(width 0.08)
@@
 	)
 	(arc
-		(start 91.2929 107.5181)
-		(mid 91.2904 107.5149)
-		(end 91.2932 107.5106)
+		(start 91.2932 107.5106)
+		(mid 91.2925 107.5121)
+		(end 91.2929 107.5181)
 		(stroke
 			(width 0.08)
@@
 	)
 	(arc
-		(start 103.171 106.7481)
-		(mid 103.1705 106.7481)
-		(end 103.17 106.7418)
+		(start 103.17 106.7418)
+		(mid 103.1741 106.7445)
+		(end 103.171 106.7481)
 		(stroke
 			(width 0.08)
